File: PCB-MP3-Player/PCB-MP3-Player.kicad_sch (KiCad schematic)
At the start: 9 parts, among them J1 Conn_01x02_Pin, J2 PCM5102A, J3 Oled, J4 Conn_01x06_Pin

Commit message: pcb changes
Parts:
- added C2, C3, C4: 100microFarad, Capacitor_THT:CP_Radial_D6.3mm_P2.50mm, symbol Device:C_Polarized
- added F2: Littelfuse 02301002H, Fuse:Fuseholder_Cylinder-5x20mm_Schurter_0031_8201_Horizontal_Open, symbol Device:Fuse
- added J5: Conn_01x02_Pin, Connector_PinSocket_2.54mm:PinSocket_1x02_P2.54mm_Vertical, symbol Connector:Conn_01x02_Pin
- added J6, J7: Conn_01x03_Pin, Connector_PinSocket_2.54mm:PinSocket_1x03_P2.54mm_Vertical, symbol Connector:Conn_01x03_Pin
- added R5, R6, R7, R8, R9: 10k, Resistor_THT:R_Axial_DIN0207_L6.3mm_D2.5mm_P7.62mm_Horizontal, symbol Device:R
- added SW1, SW2, SW3, SW4, SW5: SW_Push, Button_Switch_THT:SW_PUSH_6mm_H4.3mm, symbol Switch:SW_Push
- J4: footprint (none) -> Connector_PinSocket_2.54mm:PinSocket_1x06_P2.54mm_Vertical
Connections:
- net +3.3V: now also A1.4 (GPIO2), A1.5 (GPIO3), A1.6 (GPIO4), A1.7 (GPIO5), A1.9 (GPIO6), C2.1, C3.1, SW1.2, SW2.1, SW3.1, SW4.1, SW5.1
- net +BATT: now also C4.1, J5.1 (Pin_1)
- net -BATT: now also C4.2, J5.2 (Pin_2)
- net GND: now also C2.2, C3.2, J6.2 (Pin_2), J7.2 (Pin_2), R5.1, R6.1, R7.1, R8.1, R9.1
- net at J1.1 (Pin_1): now also F2.1; no longer D1.2 (A)
- new net: R6.2, SW2.2
- new net: R7.2, SW3.2
- new net: R5.2, SW1.1
- new net: R8.2, SW4.2
- new net: D1.2 (A), F2.2
- new net: R9.2, SW5.2
- new net L_AUDIO: J6.1 (Pin_1), J7.1 (Pin_1)
- new net R_AUDIO: J6.3 (Pin_3), J7.3 (Pin_3)
Other:
- note added: "Audio"
- note added: "Can accept 3.6v to 12v, 3.7v of battery lipo is nominal so should be ok"
- note added: "LM4881"
- note added: "Pins for PCM5102A output audio"
- moved on the sheet: D1

Commit message: connected oled
Connections:
- net at R7.2: now also SW4.2; no longer SW3.2
- net at SW1.1: now also R9.2; no longer R5.2
- net at R8.2: now also SW3.2; no longer SW4.2
- net at SW5.2: now also R5.2; no longer R9.2
Other:
- moved on the sheet: R5, R7, R8, R9
Changed lines of the file:
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@@
 		)
 	)
-	(label "BUTTON3"
-		(at 240.03 72.39 180)
+	(label "BUTTON5"
+		(at 215.9 40.64 180)
 		(effects
 			(font
@@
 		)
 	)
-	(label "BUTTON5"
-		(at 215.9 40.64 180)
+	(label "MISO"
+		(at 73.66 148.59 0)
 		(effects
 			(font
 				(size 1.27 1.27)
 			)
-			(justify right bottom)
+			(justify left bottom)
 		)
 	)
-	(label "MISO"
-		(at 73.66 148.59 0)
+	(label "BUTTON4"
+		(at 240.03 72.39 180)
 		(effects
 			(font
 				(size 1.27 1.27)
 			)
-			(justify left bottom)
+			(justify right bottom)
 		)
 	)
@@
 		)
 	)
-	(label "BUTTON4"
-		(at 237.49 57.15 180)
-		(effects
-			(font
-				(size 1.27 1.27)
-			)
-			(justify right bottom)
-		)
-	)
 	(label "L_AUDIO"
 		(at 86.36 52.07 0)
@@
 		)
 	)
+	(label "BUTTON3"
+		(at 237.49 57.15 180)
+		(effects
+			(font
+				(size 1.27 1.27)
+			)
+			(justify right bottom)
+		)
+	)
 	(label "CS"
 		(at 73.66 140.97 0)
@@
 	(symbol
 		(lib_id "Device:R")
-		(at 251.46 62.23 270)
+		(at 254 77.47 270)
 		(unit 1)
 		(body_style 1)
@@
 		(fields_autoplaced yes)
 		(property "Reference" "R7"
-			(at 251.46 55.88 90)
+			(at 254 71.12 90)
 			(show_name no)
 			(do_not_autoplace no)
@@
 		)
 		(property "Value" "10k"
-			(at 251.46 58.42 90)
+			(at 254 73.66 90)
 			(show_name no)
 			(do_not_autoplace no)
@@
 		)
 		(property "Footprint" "Resistor_THT:R_Axial_DIN0207_L6.3mm_D2.5mm_P7.62mm_Horizontal"
-			(at 251.46 60.452 90)
+			(at 254 75.692 90)
 			(hide yes)
 			(show_name no)
@@
 		)
 		(property "Datasheet" ""
-			(at 251.46 62.23 0)
+			(at 254 77.47 0)
 			(hide yes)
 			(show_name no)
@@
 		)
 		(property "Description" "Resistor"
-			(at 251.46 62.23 0)
+			(at 254 77.47 0)
 			(hide yes)
 			(show_name no)
@@
 	(symbol
 		(lib_id "Device:R")
-		(at 254 77.47 270)
+		(at 251.46 62.23 270)
 		(unit 1)
 		(body_style 1)
@@
 		(fields_autoplaced yes)
 		(property "Reference" "R8"
-			(at 254 71.12 90)
+			(at 251.46 55.88 90)
 			(show_name no)
 			(do_not_autoplace no)
@@
 		)
 		(property "Value" "10k"
-			(at 254 73.66 90)
+			(at 251.46 58.42 90)
 			(show_name no)
 			(do_not_autoplace no)
@@
 		)
 		(property "Footprint" "Resistor_THT:R_Axial_DIN0207_L6.3mm_D2.5mm_P7.62mm_Horizontal"
-			(at 254 75.692 90)
+			(at 251.46 60.452 90)
 			(hide yes)
 			(show_name no)
@@
 		)
 		(property "Datasheet" ""
-			(at 254 77.47 0)
+			(at 251.46 62.23 0)
 			(hide yes)
 			(show_name no)
@@
 		)
 		(property "Description" "Resistor"
-			(at 254 77.47 0)
+			(at 251.46 62.23 0)
 			(hide yes)
 			(show_name no)
@@
 	(symbol
 		(lib_id "Device:R")
-		(at 210.82 63.5 270)
+		(at 229.87 45.72 270)
 		(unit 1)
 		(body_style 1)
@@
 		(fields_autoplaced yes)
 		(property "Reference" "R5"
-			(at 210.82 57.15 90)
+			(at 229.87 39.37 90)
 			(show_name no)
 			(do_not_autoplace no)
@@
 		)
 		(property "Value" "10k"
-			(at 210.82 59.69 90)
+			(at 229.87 41.91 90)
 			(show_name no)
 			(do_not_autoplace no)
@@
 		)
 		(property "Footprint" "Resistor_THT:R_Axial_DIN0207_L6.3mm_D2.5mm_P7.62mm_Horizontal"
-			(at 210.82 61.722 90)
+			(at 229.87 43.942 90)
 			(hide yes)
 			(show_name no)
@@
 		)
 		(property "Datasheet" ""
-			(at 210.82 63.5 0)
+			(at 229.87 45.72 0)
 			(hide yes)
 			(show_name no)
@@
 		)
 		(property "Description" "Resistor"
-			(at 210.82 63.5 0)
+			(at 229.87 45.72 0)
 			(hide yes)
 			(show_name no)
@@
 	(symbol
 		(lib_id "Device:R")
-		(at 229.87 45.72 270)
+		(at 210.82 63.5 270)
 		(unit 1)
 		(body_style 1)
@@
 		(fields_autoplaced yes)
 		(property "Reference" "R9"
-			(at 229.87 39.37 90)
+			(at 210.82 57.15 90)
 			(show_name no)
 			(do_not_autoplace no)
@@
 		)
 		(property "Value" "10k"
-			(at 229.87 41.91 90)
+			(at 210.82 59.69 90)
 			(show_name no)
 			(do_not_autoplace no)
@@
 		)
 		(property "Footprint" "Resistor_THT:R_Axial_DIN0207_L6.3mm_D2.5mm_P7.62mm_Horizontal"
-			(at 229.87 43.942 90)
+			(at 210.82 61.722 90)
 			(hide yes)
 			(show_name no)
@@
 		)
 		(property "Datasheet" ""
-			(at 229.87 45.72 0)
+			(at 210.82 63.5 0)
 			(hide yes)
 			(show_name no)
@@
 		)
 		(property "Description" "Resistor"
-			(at 229.87 45.72 0)
+			(at 210.82 63.5 0)
 			(hide yes)
 			(show_name no)

Commit message: pcb changes
Parts:
- removed C4: 100microFarad, Capacitor_THT:CP_Radial_D6.3mm_P2.50mm, symbol Device:C_Polarized
- removed J5: Conn_01x02_Pin, Connector_PinSocket_2.54mm:PinSocket_1x02_P2.54mm_Vertical, symbol Connector:Conn_01x02_Pin
- removed J6, J7: Conn_01x03_Pin, Connector_PinSocket_2.54mm:PinSocket_1x03_P2.54mm_Vertical, symbol Connector:Conn_01x03_Pin
Connections:
- net +3.3V: now also C2.2; no longer C2.1
- net ADC_BAT: now also R4.2; no longer R4.1
- net GND: now also C1.2, C2.1, J1.2 (Pin_2), R4.1; no longer C2.2
- removed net -BATT: C1.2, J1.2 (Pin_2), R4.2
Other:
- note removed: "Audio"
- note removed: "Can accept 3.6v to 12v, 3.7v of battery lipo is nominal so should be ok"
- note removed: "LM4881"
- note removed: "Pins for PCM5102A output audio"
- moved on the sheet: C2, R4

Commit message: Devlog 7
Parts:
- J4: footprint Connector_PinSocket_2.54mm:PinSocket_1x06_P2.54mm_Vertical -> Connector_JST:JST_SHL_SM06B-SHLS-TF_1x06-1MP_P1.00mm_Horizontal
Changed lines of the file:
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@@
 			)
 		)
-		(property "Footprint" "Connector_PinSocket_2.54mm:PinSocket_1x06_P2.54mm_Vertical"
+		(property "Footprint" "Connector_JST:JST_SHL_SM06B-SHLS-TF_1x06-1MP_P1.00mm_Horizontal"
 			(at 68.58 146.05 0)
 			(hide yes)

Commit message: Adding renders, readme, etc.
Parts:
- F2: value Littelfuse 02301002H -> 520.620
- J4: footprint Connector_JST:JST_SHL_SM06B-SHLS-TF_1x06-1MP_P1.00mm_Horizontal -> Connector_JST:JST_SH_SM06B-SRSS-TB_1x06-1MP_P1.00mm_Horizontal
Changed lines of the file:
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@@
 			)
 		)
-		(property "Footprint" "Connector_JST:JST_SHL_SM06B-SHLS-TF_1x06-1MP_P1.00mm_Horizontal"
+		(property "Footprint" "Connector_JST:JST_SH_SM06B-SRSS-TB_1x06-1MP_P1.00mm_Horizontal"
 			(at 68.58 146.05 0)
 			(hide yes)
@@
 			)
 		)
-		(property "Value" "Littelfuse 02301002H"
+		(property "Value" "520.620"
 			(at 26.416 169.926 90)
 			(show_name no)
